File: EsperDNS.sch (KiCad schematic (older format))
At the start: 32 parts, among them J1 USB_B_Micro, J2 ARJM11A3, U1 AZ1117-3.3, U2 LAN8720A

Commit message: Second page finished
Parts:
- removed C1, C4: 10uF, symbol Device:C
- removed C10, C11, C12, C2, C5, C6, C7, C8, C9: 0.1uF, symbol Device:C
- removed C3: 1uF, symbol Device:C
- removed D1, D2: LED, symbol Device:LED
- removed FB1: Ferrite_Bead, symbol Device:Ferrite_Bead
- removed J1: USB_B_Micro, symbol Connector:USB_B_Micro
- removed J2: ARJM11A3, ARJM11A3, symbol ARJM11A3-009-AB-ER2-T:ARJM11A3
- removed R1, R2: 470, symbol Device:R
- removed R10, R11, R8, R9: 49.9, symbol Device:R
- removed R12, R13: 270, symbol Device:R
- removed R3, R4, R5, R6: 10K, symbol Device:R
- removed R7: 12.1K, symbol Device:R
- removed U1: AZ1117-3.3, symbol Regulator_Linear:AZ1117-3.3
- removed U2: LAN8720A, Package_DFN_QFN:QFN-24-1EP_4x4mm_P0.5mm_EP2.6x2.6mm, symbol Interface_Ethernet:LAN8720A
Connections:
- net labels removed: +3.3V, AVDD, CLKIN, CRS_DV, GND, LED1_REGOFF, LED2_nINTSEL, MDC, MDIO, RXD0, RXD1, TXD0, TXD1, TXEN, VBUS, VDDCR
- wire segments 132 -> 0
- no-connect marks 2 -> 0
Other:
- note removed: "Decoupling Caps, place near U2"
- note removed: "MODE[2:0] have internal pull-ups\nCurrently configured for:\n-10/100BASE\n-Auto-negoation enabled\n-SMI address = 0x00"
