File: programmer/programmer.sch (KiCad schematic (older format))
At the start: 21 parts, among them J1 10118192-0001LF, J2 3220-10-0100-00, Q1 2N7002ET1G, U1 TLV75533PDBV, U2 FT2232HL, U3 ASDMB-12.000MHz

Commit message: Finished version 2 of programmer, now with JTAG
Parts:
- removed Q?: 2N7002ET1G, Package_TO_SOT_SMD:SOT-23, symbol Device:Q_NMOS_GSD
- added Q2: 2N7002ET1G, Package_TO_SOT_SMD:SOT-23, symbol Device:Q_NMOS_GSD
- C1, C2, C5, C6, C7, C8, C9: LCSC Part Number (none) -> C14663
- C3: LCSC Part Number (none) -> C15849
- D1: Alternate Datasheet (none) -> https://datasheet.lcsc.com/szlcsc/Everlight-Elec-19-217-BHC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; LCSC Alternate (none) -> 19-217/BHC-ZL1M2RY/3T; LCSC Part Number (none) -> C72041
- D2: Alternate Datasheet (none) -> https://datasheet.lcsc.com/szlcsc/Everlight-Elec-19-217-GHC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; LCSC Alternate (none) -> 19-217/GHC-YR1S2/3T; LCSC Part Number (none) -> C72043
- J1: symbol programmer-rescue:10118192-0001LF-My_Symbols -> Connector:USB_B_Micro
- Q1: Alternate Datasheet (none) -> https://datasheet.lcsc.com/szlcsc/Changjiang-Electronics-Te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; LCSC Alternate (none) -> 2N7002; LCSC Part Number (none) -> C8545
- R1, R2: LCSC Part Number (none) -> C22790
- R3, R4: LCSC Part Number (none) -> C23179
- U1: Alternate Datasheet (none) -> https://datasheet.lcsc.com/szlcsc/Richtek-Tech-RT9013-33GB_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; LCSC Alternate (none) -> RT9013-33GB; LCSC Part Number (none) -> C47773
- U2: LCSC Part Number (none) -> C27882
- U3: Alternate Datasheet (none) -> https://datasheet.lcsc.com/szlcsc/Yangxing-Tech-O252012MEDH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; LCSC Alternate (none) -> O252012MEDH4MI; LCSC Part Number (none) -> C90619
Connections:
- net DTR#: now also Q2.2 (S)
- net GND: now also J1.6 (Shield); no longer J1.SH (Shield)
- net IO0: now also Q2.3 (D)
- net RTS#: now also Q2.1 (G)
Changed lines of the file:
@@
 $EndDescr
 $Comp
-L programmer-rescue:10118192-0001LF-My_Symbols J1
+L Connector:USB_B_Micro J1
 U 1 1 5DF14664
 P 1800 1900
@@
 F 3 "https://www.ftdichip.com/Support/Documents/DataSheets/ICs/DS_FT2232H.pdf" H 9100 3550 50  0001 C CNN
 F 4 "768-1347-ND" H 9100 3550 50  0001 C CNN "Digikey Part Number"
+F 5 "C27882" H 9100 3550 50  0001 C CNN "LCSC Part Number"
 	1    9100 3550
 	1    0    0    -1
@@
 F 3 "~" H 2850 1900 50  0001 C CNN
 F 4 "10V" H 2965 1809 50  0000 L CNN "Rating"
+F 5 "C14663" H 2850 1900 50  0001 C CNN "LCSC Part Number"
 	1    2850 1900
 	1    0    0    -1
@@
 F 3 "~" H 4100 1900 50  0001 C CNN
 F 4 "10V" H 4215 1809 50  0000 L CNN "Rating"
+F 5 "C14663" H 4100 1900 50  0001 C CNN "LCSC Part Number"
 	1    4100 1900
 	1    0    0    -1
@@
 F 2 "Resistor_SMD:R_0603_1608Metric" V 6930 3200 50  0001 C CNN
 F 3 "~" H 7000 3200 50  0001 C CNN
+F 4 "C22790" H 7000 3200 50  0001 C CNN "LCSC Part Number"
 	1    7000 3200
 	1    0    0    -1
@@
 F 2 "Resistor_SMD:R_0603_1608Metric" V 7430 3150 50  0001 C CNN
 F 3 "~" H 7500 3150 50  0001 C CNN
+F 4 "C22790" V 7500 3150 50  0001 C CNN "LCSC Part Number"
 	1    7500 3150
 	0    1    1    0
@@
 F 3 "https://www.onsemi.com/pub/Collateral/2N7002E-D.PDF" H 1900 3900 50  0001 C CNN
 F 4 "2N7002ET1GOSCT-ND" H 1900 3900 50  0001 C CNN "Digikey Part Number"
+F 5 "2N7002" H 1900 3900 50  0001 C CNN "LCSC Alternate"
+F 6 "https://datasheet.lcsc.com/szlcsc/Changjiang-Electronics-Tech-CJ-2N7002_C8545.pdf" H 1900 3900 50  0001 C CNN "Alternate Datasheet"
+F 7 "C8545" H 1900 3900 50  0001 C CNN "LCSC Part Number"
 	1    1900 3900
 	1    0    0    -1
@@
 F 3 "~" H 6100 2250 50  0001 C CNN
 F 4 "10V" H 6215 2159 50  0000 L CNN "Rating"
+F 5 "C14663" H 6100 2250 50  0001 C CNN "LCSC Part Number"
 	1    6100 2250
 	1    0    0    -1
@@
 F 3 "~" H 6550 2250 50  0001 C CNN
 F 4 "10V" H 6665 2159 50  0000 L CNN "Rating"
+F 5 "C14663" H 6550 2250 50  0001 C CNN "LCSC Part Number"
 	1    6550 2250
 	1    0    0    -1
@@
 F 3 "~" H 6100 1250 50  0001 C CNN
 F 4 "10V" H 6215 1159 50  0000 L CNN "Rating"
+F 5 "C14663" H 6100 1250 50  0001 C CNN "LCSC Part Number"
 	1    6100 1250
 	1    0    0    -1
@@
 F 3 "https://abracon.com/Oscillators/ASDMB.pdf" H 7250 5200 50  0001 C CNN
 F 4 "535-11180-1-ND" H 6950 4750 50  0001 C CNN "Digikey Part Number"
+F 5 "O252012MEDH4MI" H 6950 4750 50  0001 C CNN "LCSC Alternate"
+F 6 "https://datasheet.lcsc.com/szlcsc/Yangxing-Tech-O252012MEDH4MI_C90619.pdf" H 6950 4750 50  0001 C CNN "Alternate Datasheet"
+F 7 "C90619" H 6950 4750 50  0001 C CNN "LCSC Part Number"
 	1    6950 4750
 	1    0    0    -1
@@
 F 3 "https://www.we-online.de/katalog/datasheet/150060BS75000.pdf" H 2750 6300 50  0001 C CNN
 F 4 "732-4966-1-ND" V 2750 6300 50  0001 C CNN "Digikey Part Number"
+F 5 "19-217/BHC-ZL1M2RY/3T" V 2750 6300 50  0001 C CNN "LCSC Alternate"
+F 6 "https://datasheet.lcsc.com/szlcsc/Everlight-Elec-19-217-BHC-ZL1M2RY-3T_C72041.pdf" V 2750 6300 50  0001 C CNN "Alternate Datasheet"
+F 7 "C72041" V 2750 6300 50  0001 C CNN "LCSC Part Number"
 	1    2750 6300
 	0    -1   -1   0
@@
 F 3 "https://www.we-online.de/katalog/datasheet/150060GS75000.pdf" H 3200 6300 50  0001 C CNN
 F 4 "732-4971-1-ND" V 3200 6300 50  0001 C CNN "Digikey Part Number"
+F 5 "19-217/GHC-YR1S2/3T" V 3200 6300 50  0001 C CNN "LCSC Alternate"
+F 6 "https://datasheet.lcsc.com/szlcsc/Everlight-Elec-19-217-GHC-YR1S2-3T_C72043.pdf" V 3200 6300 50  0001 C CNN "Alternate Datasheet"
+F 7 "C72043" V 3200 6300 50  0001 C CNN "LCSC Part Number"
 	1    3200 6300
 	0    -1   -1   0
@@
 F 3 "~" H 2750 6700 50  0001 C CNN
 F 4 "1/10W" H 2820 6609 50  0000 L CNN "Rating"
+F 5 "C23179" H 2750 6700 50  0001 C CNN "LCSC Part Number"
 	1    2750 6700
 	1    0    0    -1
@@
 F 3 "~" H 3200 6700 50  0001 C CNN
 F 4 "1/10W" H 3270 6609 50  0000 L CNN "Rating"
+F 5 "C23179" H 3200 6700 50  0001 C CNN "LCSC Part Number"
 	1    3200 6700
 	1    0    0    -1
@@
 F 3 "~" H 7350 4200 50  0001 C CNN
 F 4 "10V" H 7465 4109 50  0000 L CNN "Rating"
+F 5 "C14663" H 7350 4200 50  0001 C CNN "LCSC Part Number"
 	1    7350 4200
 	1    0    0    -1
@@
 F 3 "~" H 7000 2250 50  0001 C CNN
 F 4 "10V" H 7115 2159 50  0000 L CNN "Rating"
+F 5 "C14663" H 7000 2250 50  0001 C CNN "LCSC Part Number"
 	1    7000 2250
 	1    0    0    -1
@@
 F 3 "http://www.ti.com/lit/ds/symlink/tlv755p.pdf" H 3550 1850 50  0001 C CNN
 F 4 "296-50411-1-ND" H 3550 1800 50  0001 C CNN "Digikey Part Number"
+F 5 "RT9013-33GB" H 3550 1800 50  0001 C CNN "LCSC Alternate"
+F 6 "https://datasheet.lcsc.com/szlcsc/Richtek-Tech-RT9013-33GB_C47773.pdf" H 3550 1800 50  0001 C CNN "Alternate Datasheet"
+F 7 "C47773" H 3550 1800 50  0001 C CNN "LCSC Part Number"
 	1    3550 1800
 	1    0    0    -1
@@
 F 3 "~" H 6550 1250 50  0001 C CNN
 F 4 "10V" H 6665 1159 50  0000 L CNN "Rating"
+F 5 "C15849" H 6550 1250 50  0001 C CNN "LCSC Part Number"
 	1    6550 1250
 	1    0    0    -1
@@
 Connection ~ 6100 2050
 $Comp
-L Device:Q_NMOS_GSD Q?
-U 1 1 5FF775F6
+L Device:Q_NMOS_GSD Q2
+U 1 1 5FF7EC17
 P 1900 4550
-F 0 "Q?" H 2104 4596 50  0000 L CNN
+F 0 "Q2" H 2104 4596 50  0000 L CNN
 F 1 "2N7002ET1G" H 2104 4505 50  0000 L CNN
 F 2 "Package_TO_SOT_SMD:SOT-23" H 2100 4650 50  0001 C CNN
 F 3 "https://www.onsemi.com/pub/Collateral/2N7002E-D.PDF" H 1900 4550 50  0001 C CNN
 F 4 "2N7002ET1GOSCT-ND" H 1900 4550 50  0001 C CNN "Digikey Part Number"
+F 5 "2N7002" H 1900 4550 50  0001 C CNN "LCSC Alternate"
+F 6 "https://datasheet.lcsc.com/szlcsc/Changjiang-Electronics-Tech-CJ-2N7002_C8545.pdf" H 1900 4550 50  0001 C CNN "Alternate Datasheet"
+F 7 "C8545" H 1900 4550 50  0001 C CNN "LCSC Part Number"
 	1    1900 4550
 	1    0    0    1
